File: Hardware/Kicad/power.sch (KiCad schematic (older format))
At the start: 37 parts

Commit message: Add files via upload
Parts:
- added R?: 0R, Libs:JUMPER_5MM, symbol R
Connections:
- net +5V: now also R?.1; no longer C?.1, C?.1, L?.2, R?.1
- new net: C?.1, C?.1, L?.2, R?.1, R?.2
